Commit message: added printed base model

File: urdf/braccio_arm.urdf (robot description, URDF)
Before this commit: robot braccio, 10 links, 9 joints
Links:
- link base_link: geometry visual mesh filename=package://endu_robotics/stl/2020_Arduino_Braccio_base.STL scale=0.001 0.001 0.001
Joints:
- joint base_joint: origin xyz=0 0 0 rpy=0 0 0 -> xyz=0 0 0.00 rpy=0 0 0
- joint shoulder_joint: origin xyz=0 -.002 0.072 rpy=-1.5708 0 0 -> xyz=0 0 0.137 rpy=-1.5708 0 0
